File: Schematic/mrf89_v0.1.sch (EAGLE design)
At the start: 22 parts, among them Q1 FC-12M, Q2 BSS84, U1 G2XX3---PW28, U5 MRF89XAM8A

Commit message: Schematic ready
Parts:
- removed BATT_IN: (no value), pinhead:PINHD-1X2
- removed C9: 100nF, rcl:C-EUC0603
- removed D2: DUOLED-GY-C, led:DUOLED-GY-C
- removed Q2: BSS84, transistor-small-signal:BSS84
- removed R4: 4k7, rcl:R-EU_R0603
- removed R5, R6: 560, rcl:R-EU_R0603
- removed S1: (no value), SparkFun:TAC_SWITCHPTH
- added C1, C2: 10pF, rcl:C-EUC0603
- added C3: 100nF, rcl:C-EUC0603
- added JP1: TC2050-Series, pinhead:PINHD-2X5
- added LED1, LED2: GREEN, led:LEDCHIP-LED0603
- C5, C6: value 10uF -> 4.7uF
- R1: value 27k 1% -> 560
- R2: value 5k6 1% -> 47k
- R3: value 47k -> 560
- U1: value G2XX3---PW28 -> MSP430FR5969; device TI_MSP430_v16:G2XX3---PW28 -> chips:MSP430FR5969
Connections:
- removed net ADC: C4.1, R1.2, R2.2, U1.2
- removed net BT_VCC: Q2.G, U1.19
- removed net IRQ0: U1.10, U5.IRQ0
- removed net IRQ1: U1.11, U5.IRQ1
- removed net LED_GREEN: R6.1, U1.15
- removed net LED_YELLOW: R5.2, U1.16
- removed net MRF_!CSCON: U1.6, U5.!CSCON
- removed net MRF_RESET: U1.18, U5.RESET
- removed net N$3: D2.AY, R5.1
- removed net N$7: D2.AG, R6.2
- removed net SHT_SCL: U1.8
- removed net SHT_SDA: U1.9
- removed net SW1: C9.1, R4.1, S1.1, S1.2, U1.13
- removed net VDD: C6.1, Q2.D
- removed net VIN: BATT_IN.2, R1.1
- new net !RST: JP1.2
- new net (NC): JP1.10
- new net DBG_UART_RXD: U1.P2.6
- new net DBG_UART_TXD: U1.P2.5
- new net GPIO_P1.1: U1.P1.1
- new net GPIO_P2.7: U1.P2.7
- new net GPIO_P3.0: U1.P3.0
- new net GPIO_P3.2: U1.P3.2
- new net MRF89_!RST: U1.P4.2
- new net MRF_!CSCONF: U1.P1.4, U5.!CSCON
- new net MRF_!RST: U5.RESET
- new net MRF_IRQ0: U1.P1.2, U5.IRQ0
- new net MRF_IRQ1: U1.P1.5, U5.IRQ1
- new net N$16: R1.2, U1.P1.0
- new net N$17: LED1.A, R1.1
- new net N$4: R3.1, U1.P4.6
- new net N$8: LED2.A, R3.2
- new net RST: R2.1, U1.RST/SBWTDIO
- new net TCK: JP1.8, U1.PJ.3/TCK
- new net TDI: JP1.5, U1.PJ.1/TDI
- new net TDO: JP1.1, U1.PJ.0/TDO
- new net TEST: JP1.6, U1.TEST/SBWTCK
- new net TMS: JP1.9, U1.PJ.2/TMS
- new net UART_CTS: U1.P4.0
- new net UART_RTS: U1.P4.1
- new net UART_RX: U1.P2.0
- new net UART_TX: U1.P2.1
- new net VCC_IN: JP1.7
- new net VCC_OUT: JP1.3
- net 3V3: now also C3.1, C4.1, C6.1, R2.2, U1.AVCC, U1.DVCC; no longer Q2.S, R3.2, R4.2, U1.1
- net GND: now also C1.2, C2.2, C3.2, JP1.4, LED1.C, LED2.C, U1.AVSS, U1.DVSS, U1.VSS_QFN; no longer BATT_IN.1, C9.2, D2.C, R2.1, S1.3, S1.4, U1.28
- net MRF_!CSDATA: now also U1.P1.3; no longer U1.5
- net N$1: now also C1.1, Q1.1, U1.LFXIN; no longer Q1.2, U1.26
- net N$2: now also C2.1, Q1.2, U1.LFXOUT; no longer Q1.1, U1.27
- net PRG_!RST: no longer R3.1, U1.24
- net PRG_TEST: no longer U1.25
- net SPI_CLK: now also U1.P2.2; no longer U1.7
- net SPI_MISO: now also U1.P1.7; no longer U1.22
- net SPI_MOSI: now also U1.P1.6; no longer U1.23
